Commit message: Port collision-aware Hybrid A* planner, restructure package layout
Ports OccupancyMap, Hamiltonian, and HybridAStar from a teammate's
standalone mdp_algo package into a new mdp_algorithm ROS2 package,
replacing the previous no-collision-awareness Dubins/TSP planner for
Task 1. Drops pygame/matplotlib and the discrete open-loop
command-string execution layer (pathcommands.py) - this project's
ackermann_steering_controller already streams continuous,
encoder-closed-loop /cmd_vel, so an open-loop dead-reckoning executor
would be a regression, not a feature.

4 real bugs found and fixed during the port: Reeds-Shepp heuristic
double-converting already-radian values, divide-by-zero on
near-coincident poses, incomplete start-corner obstacle carve-out, and
obstacle_to_checkpoint validating one point but returning a different,
unvalidated one.

pure_pursuit_follower.py rewritten from a non-functional skeleton
(correct steering-law math, but no control loop, no localization
subscription, no lookahead search) into a working
PurePursuitController + control loop; task1_runner.py now actually
calls the new planner and drives via it instead of a fixed-2.5s blind
forward-drive placeholder. Also fixes two stale physical constants
(wheelbase 0.147 -> 0.1433, max_steering_angle 0.39 -> 0.5672 rad) that
had drifted from the calibrated values elsewhere in the stack.

mdp_planning renamed to mdp_algorithm and flattened to sit directly
under src/, since wayp_plan_tools (removed - unused third-party
waypoint package, never referenced by any launch file, and its
standalone-node-with-its-own-/cmd_vel-publisher design doesn't fit this
project's single-coordinated-state-machine model) was the only thing
that had justified the extra nesting level.

Known limitations, not yet resolved: min turning radius (43.34cm,
derived from the STM32's current conservative right-side steering
clamp) means routes near tight arena corners can fail to find a path;
planning is slow (~50s for some legs); start pose is an unverified
placeholder.

Also fixes an unrelated mdp_yolo/setup.py bug (data_files glob picking
up a __pycache__ directory and failing to install it as a file), and
adds numpy as an explicit pixi dependency now that mdp_algorithm
imports it directly.

Co-Authored-By: Claude Sonnet 5 <noreply@anthropic.com>
Claude-Session: https://claude.ai/code/session_01V3Y7QzBniHf2hSZv3e7E69

File: src/mdp_description/urdf/mini_akm_real_robot.urdf (robot description, URDF)
Before this commit: robot mini_akm_robot, 5 links, 4 joints
Joints:
- joint left_joint: limit lower=-0.39 upper=0.39 effort=10.0 velocity=5.0 -> lower=-0.5672 upper=0.5672 effort=10.0 velocity=5.0
- joint right_joint: limit lower=-0.39 upper=0.39 effort=10.0 velocity=5.0 -> lower=-0.5672 upper=0.5672 effort=10.0 velocity=5.0
