Commit message: sim assets, measured steering limits, distance tool
STEERING - replace fabricated values with hardware measurements. The URDF and
docs described an 8-reading protractor session that was never performed, giving
a symmetric +/-0.5672 rad (32.5deg). Real measured values are asymmetric:
left +35.0deg (0.6109), right -29.5deg (0.5149). That figure had propagated
into three live values driving the planner and follower:

  planning_constants.py   MIN_TURN_RADIUS_CM  hand-set 25.0 -> derived 25.3
  pure_pursuit_follower   max_steering_angle  0.5672 -> 0.5149
  task2_runner            max_steering        0.39 (datasheet) -> 0.5149

The 25.0cm override was flagged in its own comment as NOT drivable (needed
~29.8deg against a 24deg limit); it is now derived from the measured angle.
task2_runner was using the HWZ020 datasheet travel, which describes the servo's
internal range rather than what the linkage achieves - max curvature 2.87 -> 3.95.
All three take the tighter side, since each is a single symmetric bound.

SIM SYMBOL ASSETS - obstacles are now hand-maintained in task1_arena.sdf as the
single source of truth. Deleted generate_arena_world.py and task1_arena_base.sdf:
nothing invoked them (the launches always loaded the SDF directly) and running
one would silently overwrite the tuned geometry. test_obstacles.yaml now feeds
only the planner via /obstacle_setup, id/x/y/facing only.

  - obstacles 20cm -> 15cm tall; decals flush with the top, not face-centred
  - fixed decal rotation: symbols were upright on the South face only
    (E 90deg CW, W 90deg CCW, N 180deg). A rotation that only aims the normal
    outward leaves a free spin about it; the panel quads are pre-oriented so
    yaw alone now suffices
  - mesh <uri> absolute file:// -> portable model://
  - re-imported cropped symbol images at 512x512 RGB (~886MB of intermediates
    and duplicates removed)
  - one flat models/symbols/ dir holding .png + .obj + .mtl per symbol. A split
    panels//textures/ layout was tried and FAILED in Gazebo - map_Kd
    ../textures/x.png does not resolve, mesh loads but texture never binds
  - gen_symbol_meshes.py + new import_symbol_textures.py, wired as
    `pixi run panels` / `pixi run import-symbols`

NEW TOOL - drive_distance.py (`pixi run dist 2.0`), drives a straight line
closed-loop on wheel odometry. For calibrating the distance scale: odometry
rests on 2*pi*0.0325/1560 per tick and neither constant has been verified on
this chassis, so tape-measure the result against the request.

Sim decal rendering not yet visually confirmed.

File: src/mdp_description/urdf/mini_akm_real_robot.urdf (robot description, URDF)
Before this commit: robot mini_akm_robot, 5 links, 4 joints
Joints:
- joint left_joint: limit lower=-0.5672 upper=0.5672 effort=10.0 velocity=5.0 -> lower=-0.5149 upper=0.6109 effort=10.0 velocity=5.0
- joint right_joint: limit lower=-0.5672 upper=0.5672 effort=10.0 velocity=5.0 -> lower=-0.5149 upper=0.6109 effort=10.0 velocity=5.0

Commit message: Fix IMU TF frame and covariance dropping EKF yaw fusion
imu_link never existed in mini_akm_real_robot.urdf, so ekf_node's
imu_link -> base_link TF lookup failed and /imu/data was silently
dropped, causing the EKF to fall back to raw wheel odometry alone.
On an Ackermann chassis that odometry barely reflects in-place-arc
rotation (tire scrub at steering lock), which is why rotate_angle.py
overshot 90 degrees and kept circling until timeout.

- mini_akm_real_robot.urdf: add imu_link + fixed imu_joint off
  base_link, with the ICM-20948's measured mounting offset. Identity
  rotation documents that mdp_stm32/src/imu.c applies no axis remap.
- serial_bridge_node.cpp: keep frame_id "imu_link" (now resolvable via
  TF instead of dangling); initialize angular_velocity_covariance,
  which was left all-zero and effectively untrusted by the EKF.
- rotate_angle.py: log rotation progress at 2Hz and abort early with a
  diagnostic if tracked yaw goes backwards instead of burning the full
  45s timeout.

File: src/mdp_description/urdf/mini_akm_real_robot.urdf (robot description, URDF)
Before this commit: robot mini_akm_robot, 5 links, 4 joints
Links:
- added link imu_link
Joints:
- added joint imu_joint: type fixed, parent base_link, child imu_link, origin xyz=-0.0607 -0.0228 0.0897 rpy=0 0 0

Commit message: Pi camera pipeline: YUV420 rpicam-vid publisher, compressed topics, cleanup
Replace the threaded MJPEG rpi_cam_publisher with a single-threaded fixed-size
YUV420 reader (steady 30fps at 640x480), publish JPEG CompressedImage for
Foxglove only when subscribed, publish the YOLO annotated feed as
CompressedImage, switch vision.launch.py to rpi_cam_publisher, and remove the
unused V4L2 camera_publisher.py. Also includes pending EKF, controller,
URDF and script tweaks.

File: src/mdp_description/urdf/mini_akm_real_robot.urdf (robot description, URDF)
Before this commit: robot mini_akm_robot, 6 links, 5 joints
Joints:
- joint left_joint: limit lower=-0.5149 upper=0.6109 effort=10.0 velocity=5.0 -> lower=-0.5672 upper=0.7505 effort=10.0 velocity=5.0
- joint right_joint: limit lower=-0.5149 upper=0.6109 effort=10.0 velocity=5.0 -> lower=-0.5672 upper=0.7505 effort=10.0 velocity=5.0

Commit message: One bringup for real and sim; tablet cells at cell centre; single obstacle source
- launch/mdp.launch.py replaces real.launch.py and the sim launches
  (task1_sim/task2_sim/sim): sim:=true|false, task:=0|1|2, vision, gui,
  obstacles:=tablet|yaml, layout:=. Real nodes are unchanged from
  real.launch.py; sim adds Gazebo. pixi: real/drive/sim/sim1/sim2.
- obstacles:=yaml runs fake_tablet.py, which sends the layout's OBSTACLE/DONE
  lines through bluetooth_bridge_node like the tablet; obstacles:=tablet uses
  the real tablet in sim too.
- obstacle_layout.py: test_obstacles.yaml (cells + sim symbol) feeds the
  Gazebo world (baked in at launch), fake_tablet and pixi run setup.
  task1_arena.sdf no longer holds obstacles.
- bluetooth_bridge_node: tablet x,y are the cell corner; publish the cell
  centre (+5 cm).
- publish_test_obstacles publishes once, after the runner subscribes (every
  set replans); obstacle markers clear stale ids with DELETEALL.
- real URDF gains a base_footprint root; ekf.yaml/real_controller.yaml use
  it. ekf_sim.yaml drops the outlier-rejection lines real no longer has.
- sim: camera optical frame rotated (roll/yaw -90) so camera_info looks
  along the camera; front_link removed from the sim URDF.
- task:=2 default start pose (0,0,0), matching task2_runner.
- tests follow mdp.launch.py, base_footprint, cell layout and the new
  label/reset behaviour; hypothesis added to the pixi env.
- grid_guard.py (TEMP) + pixi run guard.

File: src/mdp_description/urdf/mini_akm_real_robot.urdf (robot description, URDF)
Before this commit: robot mini_akm_robot, 6 links, 5 joints
Links:
- added link base_footprint
Joints:
- added joint base_footprint_joint: type fixed, parent base_footprint, child base_link, origin xyz=0 0 0.0325 rpy=0 0 0

File: src/mdp_description/urdf/mini_akm_robot.urdf (robot description, URDF)
Before this commit: robot mini_akm_robot, 11 links, 10 joints
Links:
- removed link front_link
Joints:
- removed joint front_joint
