Commit message: Complete Gazebo simulation setup: URDF joint limits, REP-103 axes, remapping, and foxglove task

File: src/mdp_description/urdf/mini_akm_robot.urdf (robot description, URDF)
Before this commit: robot mini_akm_robot, 11 links, 10 joints
Joints:
- removed joint lf_point
- added joint lf_joint: type continuous, parent left_link, child lf_link, origin xyz=0 0.0301260014087184 -0.0109999999999987 rpy=0 0 0, axis 0 1 0
- joint lb_joint: axis 0 -1 0 -> 0 1 0
- joint left_joint: axis 0 0 -1 -> 0 0 1; limit lower=-0.39 upper=0.39 effort=0 velocity=0 -> lower=-0.39 upper=0.39 effort=10.0 velocity=5.0
- joint rb_joint: axis 0 -1 0 -> 0 1 0
- joint rf_joint: axis 0 -1 0 -> 0 1 0
- joint right_joint: limit lower=-0.39 upper=0.39 effort=0 velocity=0 -> lower=-0.39 upper=0.39 effort=10.0 velocity=5.0

Commit message: feat(ros): real hardware control launch, topic_based_ros2_control URDF, and autonomy nodes

File: src/mdp_description/urdf/mini_akm_robot.urdf (robot description, URDF)
Before this commit: robot mini_akm_robot, 11 links, 10 joints
Links:
- added link base_footprint
Joints:
- added joint base_footprint_joint: type fixed, parent base_footprint, child base_link, origin xyz=0 0 0.0325 rpy=0 0 0

Commit message: feat(testing): update pure pursuit follower, planner, and launch configs for full testing

File: src/mdp_description/urdf/mini_akm_robot.urdf (robot description, URDF)
Before this commit: robot mini_akm_robot, 12 links, 11 joints
Links:
- removed link laser_link
Joints:
- removed joint laser_joint
- joint camera_joint: origin xyz=0.11365 0.00016542 0.076204 rpy=0 0 0 -> xyz=0.11365 0.00016542 0.076204 rpy=0 0 CAMERA_YAW_RAD

Commit message: Fix reverse steering in the path follower; run log/status; sim fixes
Path following (task 1 stopped reversing off the arena at the end of leg 1):
- pure_pursuit_follower: reverse curvature was negated on top of the signed
  speed, so every reverse segment steered AWAY from the path. Same
  curvature for both gears now.
- drive one same-gear segment at a time; a segment ends when its last
  point is reached or passed (no dithering over a point missed by cm).
- steer toward where the target point actually is (a "reverse" point in
  front is driven to forward, and vice versa).
- sim URDF steering limits = the real measured ones (-0.5672/+0.7505 rad);
  the datasheet +/-0.39 could not follow the planner's 22.5 cm turns.
  Offline check on the 4 planned legs: all arrive, one gear change each.

Monitoring:
- /run_log (rcl_interfaces/Log): the run's decisions - route, leg ->
  obstacle/checkpoint + forward/reverse parts, arrival error, YOLO seen,
  TARGET sent, next, finished, stop. /bt_log stays the tablet traffic;
  everything else on /rosout.
- /run_status (new mdp_interfaces/RunStatus, 2 Hz): state, leg, checkpoint,
  distance, chased waypoint, FWD/REV, cmd, scan time, YOLO counts.
- current checkpoint highlighted on /checkpoint_markers, chased waypoint on
  /path_markers. foxglove/mdp_layout.json. pixi run status/runlog/btlog.
- scan pause at each checkpoint is 3 s (scan_pause_s); the most frequent
  YOLO id in that window is sent as TARGET.

Sim/bringup:
- controller odom TF remapped to /tf (car never moved in Foxglove in sim).
- fake_tablet removed; obstacles:=yaml publishes the layout once at start.
- per-launch sim world file; pixi run bag uses --exclude-regex.
- bags/ ignored.

File: src/mdp_description/urdf/mini_akm_robot.urdf (robot description, URDF)
Before this commit: robot mini_akm_robot, 10 links, 9 joints
Joints:
- joint left_joint: limit lower=-0.39 upper=0.39 effort=10.0 velocity=5.0 -> lower=-0.5672 upper=0.7505 effort=10.0 velocity=5.0
- joint right_joint: limit lower=-0.39 upper=0.39 effort=10.0 velocity=5.0 -> lower=-0.5672 upper=0.7505 effort=10.0 velocity=5.0
