Commit message: Bringup in folders, shared runner base, one sim node; calib log; task 2 redesign
- mdp_bringup nodes split into tasks/ (task1/task2 runners on runner_base.py),
  robot/ (pose feedback, manual drive, health, bag recorder, bt monitor) and
  sim/ (sim_helpers: ultrasonic, Gazebo blocks, fake arrows in one node)
- calib: every run logs a row to calibration_log.csv (tape asked for on the
  real car, Gazebo truth in sim); straight --speed with roll-past and
  sideways drift, rotate gyro drift, turn steering delay, new calib ultrasonic
- task 2: checkpoints 1-4, ultrasonic-measured obstacles, geometric smooth
  paths, reset without restarting Gazebo, fake arrows in sim
- /run_timer: live run time above the car in Foxglove (20 Hz)
- bag_recorder: /bag/start and /bag/stop, REC buttons in Foxglove
- Foxglove layout: Task 2 tab, even button row, ultrasonic frames hidden
- task 2 carpark 60 x 50 cm inside, all walls 10 cm; HC-SR04 in the URDF
- scripts/activate_gpu.sh (already referenced by pixi.toml)

File: src/mdp_description/urdf/mdp_robot.urdf.xacro (robot description, xacro)
@@ -52,4 +52,6 @@
   <material name="picam_green"><color rgba="0.0 0.45 0.15 1"/></material>
   <material name="lens_black"><color rgba="0.05 0.05 0.05 1"/></material>
+  <material name="sonar_blue"><color rgba="0.1 0.3 0.8 1"/></material>
+  <material name="sonar_silver"><color rgba="0.75 0.75 0.78 1"/></material>
   <!-- =========================================================== body === -->
   <link name="base_footprint"/>
@@ -114,4 +116,31 @@
     <parent link="base_link"/>
     <child link="imu_link"/>
+  </joint>
+  <!-- HC-SR04 ultrasonic, front centre, looking forward (+x). Its range is
+       measured from here: task2_runner adds this offset to find the obstacle.
+       TODO measure on the car (measuring sheet row J): placed at the front of
+       the body, 50 mm above the table. -->
+  <link name="ultrasonic_link">
+    <!-- HC-SR04 look-alike: 45 x 20 mm board, two 16 mm transducers facing +x. -->
+    <visual>
+      <origin xyz="-0.0075 0 0" rpy="0 0 0"/>
+      <geometry><box size="0.0015 0.045 0.020"/></geometry>
+      <material name="sonar_blue"/>
+    </visual>
+    <visual>
+      <origin xyz="-0.001 0.013 0" rpy="0 ${pi / 2} 0"/>
+      <geometry><cylinder radius="0.008" length="0.012"/></geometry>
+      <material name="sonar_silver"/>
+    </visual>
+    <visual>
+      <origin xyz="-0.001 -0.013 0" rpy="0 ${pi / 2} 0"/>
+      <geometry><cylinder radius="0.008" length="0.012"/></geometry>
+      <material name="sonar_silver"/>
+    </visual>
+  </link>
+  <joint name="ultrasonic_joint" type="fixed">
+    <origin xyz="0.19 0 ${0.05 - wheel_radius}" rpy="0 0 0"/>
+    <parent link="base_link"/>
+    <child link="ultrasonic_link"/>
   </joint>
   <!-- Raspberry Pi Camera v2 (25 x 24 mm board, 9 mm deep). Looks along this
@@ -299,4 +328,20 @@
       </sensor>
     </gazebo>
+    <!-- The ultrasonic: a narrow lidar fan (7 beams over its ~15 deg cone).
+         sim_ultrasonic turns the nearest hit into /ultrasonic (sensor_msgs/Range),
+         the same message the real car's serial bridge publishes. -->
+    <gazebo reference="ultrasonic_link">
+      <sensor name="ultrasonic" type="gpu_lidar">
+        <topic>ultrasonic_scan</topic>
+        <update_rate>20</update_rate>
+        <lidar>
+          <scan><horizontal><samples>7</samples><resolution>1</resolution>
+            <min_angle>-0.13</min_angle><max_angle>0.13</max_angle></horizontal></scan>
+          <range><min>0.02</min><max>4.0</max><resolution>0.01</resolution></range>
+        </lidar>
+        <always_on>true</always_on>
+        <visualize>false</visualize>
+      </sensor>
+    </gazebo>
     <gazebo reference="camera_link">
       <sensor name="camera" type="camera">

Commit message: Real car: calibration, gyro bias re-measured on every pose reset, smooth LQR path following with safe arrivals and off-path stop, 5-block layout

File: src/mdp_description/urdf/mdp_robot.urdf.xacro (robot description, xacro)
@@ -29,7 +29,11 @@
   <xacro:property name="rear_track" value="0.162"/>    <!-- wheel centre to centre -->
   <xacro:property name="front_track" value="0.164"/>
-  <!-- 66.2 mm tyre: what the tyres roll like (tape vs odometry, 4 x 2.0 m: the
-       car went 1.018x what 65 mm predicts). Front and rear the same tyre. -->
-  <xacro:property name="wheel_radius" value="0.0331"/>
+  <!-- 66.6 mm tyre: what the tyres roll like, from tape vs odometry. First
+       4 x 2.0 m: the car went 1.018x what 65 mm predicts -> 0.0331. Re-measured
+       2026-10-01 (calibration_log.csv, calib straight 2.0 at 0.15 and 0.41 m/s):
+       4 of 5 runs went 1.005-1.0085x odometry, mean 1.0068 -> 0.0333. The fifth
+       (0.980, and 15 cm sideways) was a bad run, left out. Front and rear the
+       same tyre. -->
+  <xacro:property name="wheel_radius" value="0.0333"/>
   <!-- Front wheel centre sits this far outboard of its steering pivot, and the
        pivot this far above the wheel centre (CAD). -->

Commit message: Task 1: fix the position at each scan stop with the two left IRs
At a scan stop the runner waits for 3 readings per IR (max 1.5 s); if only
one IR sees the block's image side it creeps straight towards it until both
do (the beam crossing the block edge gives the along-face position), sets
the EKF pose from the edge and the median IR gap (heading kept), drives
straight to level base_link with the block centre, and replans the next leg
during the scan if the car is more than 2 cm off its start.

- tasks/ir_pose_fix.py: the geometry (no ROS) + test/test_ir_pose_fix.py
- task1_runner: ir_stop_step / creep / apply_ir_fix (robot_localization
  set_pose service, so no RESET); switch: parameter ir_pose_fix
- navigation.yaml: follower.creep_linear_vel 0.05 m/s
- URDF: ir_link / ir2_link 4 cm either side of the rear axle on the left
  (placeholders, TODO measure); camera at the rear axle above the right
  rear wheel (new mount)
- sim: sim/ir.py publishes /ir, /ir2 from gpu_lidar stand-ins

Sim 2026-10-04 (5 obstacles, natural drift): estimate error after each
scan 2.6-6.4 cm without, 0.3-2.0 cm with; along-face stop error up to
5.7 cm without, <=2.4 cm with; run 52 s -> 59 s.

File: src/mdp_description/urdf/mdp_robot.urdf.xacro (robot description, xacro)
@@ -148,9 +148,35 @@
     <child link="ultrasonic_link"/>
   </joint>
+  <!-- Two Sharp GP2Y0A21YK IRs on the LEFT side, looking left (+y), one ahead of
+       and one behind the rear axle: a scan checkpoint puts base_link (the rear
+       axle) square in front of the block's centre, so at the stop both see
+       its 10 cm face, and task1_runner corrects the car's position against
+       the block (tasks/ir_pose_fix.py). /ir = ir_link (front), /ir2 = ir2_link
+       (rear). Their ranges are measured from here. TODO measure on the car:
+       placed 40 mm either side of the rear axle, at the left edge of the body,
+       90 mm above the table (clear of the wheels; the blocks are 15 cm tall). -->
+  <xacro:macro name="sharp_ir" params="name x">
+    <link name="${name}_link">
+      <visual>
+        <origin xyz="-0.0065 0 0" rpy="0 0 0"/>
+        <geometry><box size="0.013 0.0295 0.0135"/></geometry>
+        <material name="lens_black"/>
+      </visual>
+    </link>
+    <joint name="${name}_joint" type="fixed">
+      <origin xyz="${x} 0.085 ${0.09 - wheel_radius}" rpy="0 0 ${pi / 2}"/>
+      <parent link="base_link"/>
+      <child link="${name}_link"/>
+    </joint>
+  </xacro:macro>
+  <xacro:sharp_ir name="ir" x="0.04"/>
+  <xacro:sharp_ir name="ir2" x="-0.04"/>
   <!-- Raspberry Pi Camera v2 (25 x 24 mm board, 9 mm deep). Looks along this
-       link's +x; camera_yaw turns it (task 1: left). Placed 2026-09-28 at the
-       middle of the chassis on the centre line, 84 mm ahead of the rear axle
-       (the body runs 31 mm behind to 199 mm ahead), at the CAD mount's height
-       (60 mm above the axle). TODO measure once mounted (sheet rows H1-H5). -->
+       link's +x; camera_yaw turns it (task 1: left). On the 3D-printed mount
+       above the right rear wheel (2026-10-03): in line with the rear axle,
+       so base_link - which a scan checkpoint puts square in front of the
+       block's centre - and the camera face the image together. Height still
+       the CAD mount's (60 mm above the axle); the print puts the lens ~80 mm
+       above the STM32. TODO measure once mounted (sheet rows H1-H5). -->
   <link name="camera_link">
     <visual>
@@ -173,5 +199,5 @@
   </link>
   <joint name="camera_joint" type="fixed">
-    <origin xyz="0.084 0 ${cad_z + 0.076204}" rpy="0 0 $(arg camera_yaw)"/>
+    <origin xyz="0 ${-rear_track / 2} ${cad_z + 0.076204}" rpy="0 0 $(arg camera_yaw)"/>
     <parent link="base_link"/>
     <child link="camera_link"/>
@@ -348,4 +374,24 @@
       </sensor>
     </gazebo>
+    <!-- The IRs: a 3-beam lidar each (the Sharp's beam is narrow, ~2 deg).
+         sim_helpers turns them into /ir and /ir2 (sim/ir.py), as the bridge.
+         25 Hz: what the Sharp gives (one reading per ~38 ms). -->
+    <xacro:macro name="sharp_ir_sensor" params="name">
+      <gazebo reference="${name}_link">
+        <sensor name="${name}" type="gpu_lidar">
+          <topic>${name}_scan</topic>
+          <update_rate>25</update_rate>
+          <lidar>
+            <scan><horizontal><samples>3</samples><resolution>1</resolution>
+              <min_angle>-0.017</min_angle><max_angle>0.017</max_angle></horizontal></scan>
+            <range><min>0.02</min><max>1.0</max><resolution>0.001</resolution></range>
+          </lidar>
+          <always_on>true</always_on>
+          <visualize>false</visualize>
+        </sensor>
+      </gazebo>
+    </xacro:macro>
+    <xacro:sharp_ir_sensor name="ir"/>
+    <xacro:sharp_ir_sensor name="ir2"/>
     <gazebo reference="camera_link">
       <sensor name="camera" type="camera">

Commit message: URDF: measured IR positions - IR2 (/ir2) 42 mm ahead of the rear axle, IR1 (/ir) 30 mm behind, both 62 mm left

File: src/mdp_description/urdf/mdp_robot.urdf.xacro (robot description, xacro)
@@ -152,8 +152,10 @@
        axle) square in front of the block's centre, so at the stop both see
        its 10 cm face, and task1_runner corrects the car's position against
-       the block (tasks/ir_pose_fix.py). /ir = ir_link (front), /ir2 = ir2_link
-       (rear). Their ranges are measured from here. TODO measure on the car:
-       placed 40 mm either side of the rear axle, at the left edge of the body,
-       90 mm above the table (clear of the wheels; the blocks are 15 cm tall). -->
+       the block (tasks/ir_pose_fix.py; it takes whichever is further forward as
+       the front one). Their ranges are measured from here.
+       Measured on the car 2026-10-07: IR2 (/ir2, ir2_link) 42 mm AHEAD of the rear
+       axle, IR1 (/ir, ir_link) 72 mm behind it = 30 mm BEHIND the rear axle.
+       Both faces 62 mm left of the centre line (base_link y). Height 90 mm above
+       the table (not measured; only needs to clear the left rear tyre, top ~66 mm). -->
   <xacro:macro name="sharp_ir" params="name x">
     <link name="${name}_link">
@@ -165,11 +167,11 @@
     </link>
     <joint name="${name}_joint" type="fixed">
-      <origin xyz="${x} 0.085 ${0.09 - wheel_radius}" rpy="0 0 ${pi / 2}"/>
+      <origin xyz="${x} 0.062 ${0.09 - wheel_radius}" rpy="0 0 ${pi / 2}"/>
       <parent link="base_link"/>
       <child link="${name}_link"/>
     </joint>
   </xacro:macro>
-  <xacro:sharp_ir name="ir" x="0.04"/>
-  <xacro:sharp_ir name="ir2" x="-0.04"/>
+  <xacro:sharp_ir name="ir" x="-0.030"/>    <!-- IR1, /ir: the rear one -->
+  <xacro:sharp_ir name="ir2" x="0.042"/>    <!-- IR2, /ir2: the front one -->
   <!-- Raspberry Pi Camera v2 (25 x 24 mm board, 9 mm deep). Looks along this
        link's +x; camera_yaw turns it (task 1: left). On the 3D-printed mount

Commit message: IR: measured positions in the URDF; curves from calib ir runs on the car

File: src/mdp_description/urdf/mdp_robot.urdf.xacro (robot description, xacro)
@@ -152,8 +152,10 @@
        axle) square in front of the block's centre, so at the stop both see
        its 10 cm face, and task1_runner corrects the car's position against
-       the block (tasks/ir_pose_fix.py). /ir = ir_link (front), /ir2 = ir2_link
-       (rear). Their ranges are measured from here. TODO measure on the car:
-       placed 40 mm either side of the rear axle, at the left edge of the body,
-       90 mm above the table (clear of the wheels; the blocks are 15 cm tall). -->
+       the block (tasks/ir_pose_fix.py; it takes whichever is further forward as
+       the front one). Their ranges are measured from here.
+       Measured on the car 2026-10-07: IR2 (/ir2, ir2_link) 41 mm AHEAD of the rear
+       axle, IR1 (/ir, ir_link) 72.5 mm behind it = 31.5 mm BEHIND the rear axle.
+       Both faces 62 mm left of the centre line (base_link y). Height 90 mm above
+       the table (not measured; only needs to clear the left rear tyre, top ~66 mm). -->
   <xacro:macro name="sharp_ir" params="name x">
     <link name="${name}_link">
@@ -165,11 +167,11 @@
     </link>
     <joint name="${name}_joint" type="fixed">
-      <origin xyz="${x} 0.085 ${0.09 - wheel_radius}" rpy="0 0 ${pi / 2}"/>
+      <origin xyz="${x} 0.062 ${0.09 - wheel_radius}" rpy="0 0 ${pi / 2}"/>
       <parent link="base_link"/>
       <child link="${name}_link"/>
     </joint>
   </xacro:macro>
-  <xacro:sharp_ir name="ir" x="0.04"/>
-  <xacro:sharp_ir name="ir2" x="-0.04"/>
+  <xacro:sharp_ir name="ir" x="-0.0315"/>   <!-- IR1, /ir: the rear one -->
+  <xacro:sharp_ir name="ir2" x="0.041"/>    <!-- IR2, /ir2: the front one -->
   <!-- Raspberry Pi Camera v2 (25 x 24 mm board, 9 mm deep). Looks along this
        link's +x; camera_yaw turns it (task 1: left). On the 3D-printed mount

Commit message: URDF: front wheels drawn on the real car (fixed), ultrasonic on top of the chassis, IRs upright, camera measured - 175 mm up, 55 mm right

File: src/mdp_description/urdf/mdp_robot.urdf.xacro (robot description, xacro)
@@ -123,6 +123,6 @@
   <!-- HC-SR04 ultrasonic, front centre, looking forward (+x). Its range is
        measured from here: task2_runner adds this offset to find the obstacle.
-       TODO measure on the car (measuring sheet row J): placed at the front of
-       the body, 50 mm above the table. -->
+       Right on top of the chassis at its front (2026-10-08): the chassis top is
+       69 mm above the table (base_link mesh), the 20 mm board's centre 79 mm. -->
   <link name="ultrasonic_link">
     <!-- HC-SR04 look-alike: 45 x 20 mm board, two 16 mm transducers facing +x. -->
@@ -144,5 +144,5 @@
   </link>
   <joint name="ultrasonic_joint" type="fixed">
-    <origin xyz="0.19 0 ${0.05 - wheel_radius}" rpy="0 0 0"/>
+    <origin xyz="0.19 0 ${0.079 - wheel_radius}" rpy="0 0 0"/>
     <parent link="base_link"/>
     <child link="ultrasonic_link"/>
@@ -162,5 +162,6 @@
       <visual>
         <origin xyz="-0.0065 0 0" rpy="0 0 0"/>
-        <geometry><box size="0.013 0.0295 0.0135"/></geometry>
+        <!-- 13 deep x 13.5 wide x 29.5 mm tall: mounted upright (2026-10-08). -->
+        <geometry><box size="0.013 0.0135 0.0295"/></geometry>
         <material name="lens_black"/>
       </visual>
@@ -178,7 +179,7 @@
        above the right rear wheel (2026-10-03): in line with the rear axle,
        so base_link - which a scan checkpoint puts square in front of the
-       block's centre - and the camera face the image together. Height still
-       the CAD mount's (60 mm above the axle); the print puts the lens ~80 mm
-       above the STM32. TODO measure once mounted (sheet rows H1-H5). -->
+       block's centre - and the camera face the image together. Measured on the
+       car 2026-10-08: the lens 175 mm above the table, 55 mm right of the centre
+       line. -->
   <link name="camera_link">
     <visual>
@@ -201,5 +202,5 @@
   </link>
   <joint name="camera_joint" type="fixed">
-    <origin xyz="0 ${-rear_track / 2} ${cad_z + 0.076204}" rpy="0 0 $(arg camera_yaw)"/>
+    <origin xyz="0 -0.055 ${0.175 - wheel_radius}" rpy="0 0 $(arg camera_yaw)"/>
     <parent link="base_link"/>
     <child link="camera_link"/>
@@ -247,6 +248,5 @@
   <xacro:rear_wheel side="r" sign="-1"/>
   <!-- Front: steering knuckle (left_link / right_link, both at the same angle -
-       one servo and a tie rod), then the free-spinning wheel (sim only: the
-       real car has no front encoders). -->
+       one servo and a tie rod), then the free-spinning wheel. -->
   <xacro:macro name="front_wheel" params="side knuckle sign">
     <link name="${knuckle}_link">
@@ -274,13 +274,13 @@
       <limit lower="${-steer_right}" upper="${steer_left}" effort="10.0" velocity="5.0"/>
     </joint>
-    <xacro:if value="${sim}">
-      <xacro:tyre name="${side}f_link" mesh_name="${side}f_link" width="0.026" y_offset="${-sign * 0.00045}"/>
-      <joint name="${side}f_joint" type="continuous">
-        <origin xyz="0 ${sign * knuckle_out} ${-knuckle_up}" rpy="0 0 0"/>
-        <parent link="${knuckle}_link"/>
-        <child link="${side}f_link"/>
-        <axis xyz="0 1 0"/>
-      </joint>
-    </xacro:if>
+    <xacro:tyre name="${side}f_link" mesh_name="${side}f_link" width="0.026" y_offset="${-sign * 0.00045}"/>
+    <!-- Sim: spins (Gazebo reports it). Real car: no front encoders, so nothing
+         would publish its angle - fixed, just drawn (it steers with the knuckle). -->
+    <joint name="${side}f_joint" type="${'continuous' if sim else 'fixed'}">
+      <origin xyz="0 ${sign * knuckle_out} ${-knuckle_up}" rpy="0 0 0"/>
+      <parent link="${knuckle}_link"/>
+      <child link="${side}f_link"/>
+      <xacro:if value="${sim}"><axis xyz="0 1 0"/></xacro:if>
+    </joint>
   </xacro:macro>
   <xacro:front_wheel side="l" knuckle="left" sign="1"/>

Commit message: Task 2 (trial): no stop at checkpoint 1 (roll on toward the centre while arrow 2 / the bar is unknown, nearer end at 60 cm), IR fixes at obstacle 1's side and the bar's ends (pose-lag compensated, two edges); task 2 URDF puts the IRs at the front wheels

File: src/mdp_description/urdf/mdp_robot.urdf.xacro (robot description, xacro)
@@ -22,4 +22,5 @@
   <xacro:arg name="sim" default="false"/>
   <xacro:arg name="camera_yaw" default="0.0"/>        <!-- task 1: 1.5708 (camera looks LEFT) -->
+  <xacro:arg name="task" default="1"/>                <!-- 2: the IRs move to the front wheels (sharp_ir) -->
   <xacro:arg name="controller_config" default=""/>    <!-- sim: absolute path of controller.yaml -->
   <xacro:property name="sim" value="$(arg sim)"/>
@@ -158,5 +159,5 @@
        Both faces 62 mm left of the centre line (base_link y). Height 90 mm above
        the table (not measured; only needs to clear the left rear tyre, top ~66 mm). -->
-  <xacro:macro name="sharp_ir" params="name x">
+  <xacro:macro name="sharp_ir" params="name x y:=0.062 yaw:=${pi / 2}">
     <link name="${name}_link">
       <visual>
@@ -168,11 +169,20 @@
     </link>
     <joint name="${name}_joint" type="fixed">
-      <origin xyz="${x} 0.062 ${0.09 - wheel_radius}" rpy="0 0 ${pi / 2}"/>
+      <origin xyz="${x} ${y} ${0.09 - wheel_radius}" rpy="0 0 ${yaw}"/>
       <parent link="base_link"/>
       <child link="${name}_link"/>
     </joint>
   </xacro:macro>
-  <xacro:sharp_ir name="ir" x="-0.0315"/>   <!-- IR1, /ir: the rear one -->
-  <xacro:sharp_ir name="ir2" x="0.041"/>    <!-- IR2, /ir2: the front one -->
+  <xacro:if value="${'$(arg task)' != '2'}">
+    <xacro:sharp_ir name="ir" x="-0.0315"/>   <!-- IR1, /ir: the rear one -->
+    <xacro:sharp_ir name="ir2" x="0.041"/>    <!-- IR2, /ir2: the front one -->
+  </xacro:if>
+  <!-- Task 2 (2026-10-10, not measured yet): one IR each side at the front axle, looking
+       out - IR1 right, IR2 left - for the sides of obstacle 1 and the bar's ends.
+       Same height and 62 mm out as task 1; the beam passes over the front tyres. -->
+  <xacro:if value="${'$(arg task)' == '2'}">
+    <xacro:sharp_ir name="ir" x="${wheelbase}" y="-0.062" yaw="${-pi / 2}"/>   <!-- IR1, /ir: right -->
+    <xacro:sharp_ir name="ir2" x="${wheelbase}" y="0.062"/>                    <!-- IR2, /ir2: left -->
+  </xacro:if>
   <!-- Raspberry Pi Camera v2 (25 x 24 mm board, 9 mm deep). Looks along this
        link's +x; camera_yaw turns it (task 1: left). On the 3D-printed mount

Commit message: Task 2 IR fixes: a runner-side offset aligned by stamps, 'out' only at the bar's ends; camera at the front on the centre line

File: src/mdp_description/urdf/mdp_robot.urdf.xacro (robot description, xacro)
@@ -211,6 +211,9 @@
     </xacro:if>
   </link>
+  <!-- Task 2 (2026-10-10, not measured yet): at the front of the car on the centre
+       line, same height - looking ahead at the arrows. -->
+  <xacro:property name="camera_xy" value="${'0.19 0' if '$(arg task)' == '2' else '0 -0.055'}"/>
   <joint name="camera_joint" type="fixed">
-    <origin xyz="0 -0.055 ${0.175 - wheel_radius}" rpy="0 0 $(arg camera_yaw)"/>
+    <origin xyz="${camera_xy} ${0.175 - wheel_radius}" rpy="0 0 $(arg camera_yaw)"/>
     <parent link="base_link"/>
     <child link="camera_link"/>
