Commit message: URDF, measured 2026-10-14: ultrasonic transducers 13 mm past the chassis front = 212 mm ahead of the rear axle (was 190: task 2's obstacle distances 22 mm short); task 2 IRs 50 mm behind the chassis front (149 mm), faces 13 mm out from its 80 mm front = 53 mm each side (was 62 at the front axle, not measured)

File: src/mdp_description/urdf/mdp_robot.urdf.xacro (robot description, xacro)
@@ -125,5 +125,8 @@
        measured from here: task2_runner adds this offset to find the obstacle.
        Right on top of the chassis at its front (2026-10-08): the chassis top is
-       69 mm above the table (base_link mesh), the 20 mm board's centre 79 mm. -->
+       69 mm above the table (base_link mesh), the 20 mm board's centre 79 mm.
+       The transducers' fronts (this link) stick out 13 mm past the chassis
+       front, which is 199 mm ahead of the rear axle (measured 2026-10-14; was
+       190 mm, 22 mm short - every obstacle distance was off by that). -->
   <link name="ultrasonic_link">
     <!-- HC-SR04 look-alike: 45 x 20 mm board, two 16 mm transducers facing +x. -->
@@ -145,5 +148,5 @@
   </link>
   <joint name="ultrasonic_joint" type="fixed">
-    <origin xyz="0.19 0 ${0.079 - wheel_radius}" rpy="0 0 0"/>
+    <origin xyz="${0.199 + 0.013} 0 ${0.079 - wheel_radius}" rpy="0 0 0"/>
     <parent link="base_link"/>
     <child link="ultrasonic_link"/>
@@ -178,10 +181,12 @@
     <xacro:sharp_ir name="ir2" x="0.041"/>    <!-- IR2, /ir2: the front one -->
   </xacro:if>
-  <!-- Task 2 (2026-10-10, not measured yet): one IR each side at the front axle, looking
-       out - IR1 right, IR2 left - for the sides of obstacle 1 and the bar's ends.
-       Same height and 62 mm out as task 1; the beam passes over the front tyres. -->
+  <!-- Task 2: one IR each side near the front, looking out - IR1 right, IR2 left -
+       for the sides of obstacle 1 and the bar's ends. Measured on the car
+       2026-10-14: centres 50 mm behind the chassis front (199 mm ahead of the
+       rear axle), faces 13 mm out from the chassis' 80 mm wide front (CAD:
+       40 mm each side). Height as task 1, not measured. -->
   <xacro:if value="${'$(arg task)' == '2'}">
-    <xacro:sharp_ir name="ir" x="${wheelbase}" y="-0.062" yaw="${-pi / 2}"/>   <!-- IR1, /ir: right -->
-    <xacro:sharp_ir name="ir2" x="${wheelbase}" y="0.062"/>                    <!-- IR2, /ir2: left -->
+    <xacro:sharp_ir name="ir" x="${0.199 - 0.050}" y="${-(0.040 + 0.013)}" yaw="${-pi / 2}"/>   <!-- IR1, /ir: right -->
+    <xacro:sharp_ir name="ir2" x="${0.199 - 0.050}" y="${0.040 + 0.013}"/>                      <!-- IR2, /ir2: left -->
   </xacro:if>
   <!-- Raspberry Pi Camera v2 (25 x 24 mm board, 9 mm deep). Looks along this

Commit message: URDF task 2, measured 2026-10-14: camera lens 28 mm behind the chassis front (171 mm ahead of the rear axle), 150 mm above the table, centre line; IRs lying on their sides (horizontal)

File: src/mdp_description/urdf/mdp_robot.urdf.xacro (robot description, xacro)
@@ -162,10 +162,12 @@
        Both faces 62 mm left of the centre line (base_link y). Height 90 mm above
        the table (not measured; only needs to clear the left rear tyre, top ~66 mm). -->
-  <xacro:macro name="sharp_ir" params="name x y:=0.062 yaw:=${pi / 2}">
+  <xacro:macro name="sharp_ir" params="name x y:=0.062 yaw:=${pi / 2} lying:=false">
     <link name="${name}_link">
       <visual>
         <origin xyz="-0.0065 0 0" rpy="0 0 0"/>
-        <!-- 13 deep x 13.5 wide x 29.5 mm tall: mounted upright (2026-10-08). -->
-        <geometry><box size="0.013 0.0135 0.0295"/></geometry>
+        <!-- 13 deep x 13.5 wide x 29.5 mm tall: mounted upright (task 1, 2026-10-08);
+             lying: on its side, 29.5 wide x 13.5 tall (task 2, 2026-10-14). -->
+        <xacro:if value="${lying}"><geometry><box size="0.013 0.0295 0.0135"/></geometry></xacro:if>
+        <xacro:unless value="${lying}"><geometry><box size="0.013 0.0135 0.0295"/></geometry></xacro:unless>
         <material name="lens_black"/>
       </visual>
@@ -185,8 +187,9 @@
        2026-10-14: centres 50 mm behind the chassis front (199 mm ahead of the
        rear axle), faces 13 mm out from the chassis' 80 mm wide front (CAD:
-       40 mm each side). Height as task 1, not measured. -->
+       40 mm each side), lying on their sides (horizontal). Height as task 1,
+       not measured. -->
   <xacro:if value="${'$(arg task)' == '2'}">
-    <xacro:sharp_ir name="ir" x="${0.199 - 0.050}" y="${-(0.040 + 0.013)}" yaw="${-pi / 2}"/>   <!-- IR1, /ir: right -->
-    <xacro:sharp_ir name="ir2" x="${0.199 - 0.050}" y="${0.040 + 0.013}"/>                      <!-- IR2, /ir2: left -->
+    <xacro:sharp_ir name="ir" x="${0.199 - 0.050}" y="${-(0.040 + 0.013)}" yaw="${-pi / 2}" lying="true"/>   <!-- IR1, /ir: right -->
+    <xacro:sharp_ir name="ir2" x="${0.199 - 0.050}" y="${0.040 + 0.013}" lying="true"/>                      <!-- IR2, /ir2: left -->
   </xacro:if>
   <!-- Raspberry Pi Camera v2 (25 x 24 mm board, 9 mm deep). Looks along this
@@ -216,9 +219,11 @@
     </xacro:if>
   </link>
-  <!-- Task 2 (2026-10-10, not measured yet): at the front of the car on the centre
-       line, same height - looking ahead at the arrows. -->
-  <xacro:property name="camera_xy" value="${'0.19 0' if '$(arg task)' == '2' else '0 -0.055'}"/>
+  <!-- Task 2: at the front on the centre line, looking ahead at the arrows.
+       Measured on the car 2026-10-14: the lens 28 mm behind the chassis front
+       (199 mm ahead of the rear axle) and 150 mm above the table. -->
+  <xacro:property name="camera_xyz"
+                  value="${'%s 0 %s' % (0.199 - 0.028, 0.150 - wheel_radius) if '$(arg task)' == '2' else '0 -0.055 %s' % (0.175 - wheel_radius)}"/>
   <joint name="camera_joint" type="fixed">
-    <origin xyz="${camera_xy} ${0.175 - wheel_radius}" rpy="0 0 $(arg camera_yaw)"/>
+    <origin xyz="${camera_xyz}" rpy="0 0 $(arg camera_yaw)"/>
     <parent link="base_link"/>
     <child link="camera_link"/>

Commit message: Task 2 mounts measured (URDF ultrasonic, camera, IRs); IR curves only in bridges.yaml, recalibrated (IR1 [6.69, 1.111], IR2 [6.95, 1.077]); calib ir waits for Enter, break between the sensors

File: src/mdp_description/urdf/mdp_robot.urdf.xacro (robot description, xacro)
@@ -125,5 +125,8 @@
        measured from here: task2_runner adds this offset to find the obstacle.
        Right on top of the chassis at its front (2026-10-08): the chassis top is
-       69 mm above the table (base_link mesh), the 20 mm board's centre 79 mm. -->
+       69 mm above the table (base_link mesh), the 20 mm board's centre 79 mm.
+       The transducers' fronts (this link) stick out 13 mm past the chassis
+       front, which is 199 mm ahead of the rear axle (measured 2026-10-14; was
+       190 mm, 22 mm short - every obstacle distance was off by that). -->
   <link name="ultrasonic_link">
     <!-- HC-SR04 look-alike: 45 x 20 mm board, two 16 mm transducers facing +x. -->
@@ -145,5 +148,5 @@
   </link>
   <joint name="ultrasonic_joint" type="fixed">
-    <origin xyz="0.19 0 ${0.079 - wheel_radius}" rpy="0 0 0"/>
+    <origin xyz="${0.199 + 0.013} 0 ${0.079 - wheel_radius}" rpy="0 0 0"/>
     <parent link="base_link"/>
     <child link="ultrasonic_link"/>
@@ -159,10 +162,12 @@
        Both faces 62 mm left of the centre line (base_link y). Height 90 mm above
        the table (not measured; only needs to clear the left rear tyre, top ~66 mm). -->
-  <xacro:macro name="sharp_ir" params="name x y:=0.062 yaw:=${pi / 2}">
+  <xacro:macro name="sharp_ir" params="name x y:=0.062 yaw:=${pi / 2} lying:=false">
     <link name="${name}_link">
       <visual>
         <origin xyz="-0.0065 0 0" rpy="0 0 0"/>
-        <!-- 13 deep x 13.5 wide x 29.5 mm tall: mounted upright (2026-10-08). -->
-        <geometry><box size="0.013 0.0135 0.0295"/></geometry>
+        <!-- 13 deep x 13.5 wide x 29.5 mm tall: mounted upright (task 1, 2026-10-08);
+             lying: on its side, 29.5 wide x 13.5 tall (task 2, 2026-10-14). -->
+        <xacro:if value="${lying}"><geometry><box size="0.013 0.0295 0.0135"/></geometry></xacro:if>
+        <xacro:unless value="${lying}"><geometry><box size="0.013 0.0135 0.0295"/></geometry></xacro:unless>
         <material name="lens_black"/>
       </visual>
@@ -178,10 +183,13 @@
     <xacro:sharp_ir name="ir2" x="0.041"/>    <!-- IR2, /ir2: the front one -->
   </xacro:if>
-  <!-- Task 2 (2026-10-10, not measured yet): one IR each side at the front axle, looking
-       out - IR1 right, IR2 left - for the sides of obstacle 1 and the bar's ends.
-       Same height and 62 mm out as task 1; the beam passes over the front tyres. -->
+  <!-- Task 2: one IR each side near the front, looking out - IR1 right, IR2 left -
+       for the sides of obstacle 1 and the bar's ends. Measured on the car
+       2026-10-14: centres 50 mm behind the chassis front (199 mm ahead of the
+       rear axle), faces 13 mm out from the chassis' 80 mm wide front (CAD:
+       40 mm each side), lying on their sides (horizontal). Height as task 1,
+       not measured. -->
   <xacro:if value="${'$(arg task)' == '2'}">
-    <xacro:sharp_ir name="ir" x="${wheelbase}" y="-0.062" yaw="${-pi / 2}"/>   <!-- IR1, /ir: right -->
-    <xacro:sharp_ir name="ir2" x="${wheelbase}" y="0.062"/>                    <!-- IR2, /ir2: left -->
+    <xacro:sharp_ir name="ir" x="${0.199 - 0.050}" y="${-(0.040 + 0.013)}" yaw="${-pi / 2}" lying="true"/>   <!-- IR1, /ir: right -->
+    <xacro:sharp_ir name="ir2" x="${0.199 - 0.050}" y="${0.040 + 0.013}" lying="true"/>                      <!-- IR2, /ir2: left -->
   </xacro:if>
   <!-- Raspberry Pi Camera v2 (25 x 24 mm board, 9 mm deep). Looks along this
@@ -211,9 +219,11 @@
     </xacro:if>
   </link>
-  <!-- Task 2 (2026-10-10, not measured yet): at the front of the car on the centre
-       line, same height - looking ahead at the arrows. -->
-  <xacro:property name="camera_xy" value="${'0.19 0' if '$(arg task)' == '2' else '0 -0.055'}"/>
+  <!-- Task 2: at the front on the centre line, looking ahead at the arrows.
+       Measured on the car 2026-10-14: the lens 28 mm behind the chassis front
+       (199 mm ahead of the rear axle) and 150 mm above the table. -->
+  <xacro:property name="camera_xyz"
+                  value="${'%s 0 %s' % (0.199 - 0.028, 0.150 - wheel_radius) if '$(arg task)' == '2' else '0 -0.055 %s' % (0.175 - wheel_radius)}"/>
   <joint name="camera_joint" type="fixed">
-    <origin xyz="${camera_xy} ${0.175 - wheel_radius}" rpy="0 0 $(arg camera_yaw)"/>
+    <origin xyz="${camera_xyz}" rpy="0 0 $(arg camera_yaw)"/>
     <parent link="base_link"/>
     <child link="camera_link"/>
